Commit message: 使用新的imu到lidar的tf，base_link固定到lidar，新增base_frame,base_frame与imu固定

File: launch/include/config/robot.urdf.xacro (robot description, xacro)
@@ -2,26 +2,26 @@
 <robot name="lio" xmlns:xacro="http://tixiaoshan.github.io/">
   <xacro:property name="PI" value="3.1415926535897931" />
-  <link name="chassis_link"></link>
+  <link name="base_frame"></link>
   <link name="base_link"></link>
   <joint name="base_link_joint" type="fixed">
     <parent link="base_link"/>
-    <child link="chassis_link" />
-    <origin xyz="0 0 0" rpy="0 0 0" />
+    <child link="base_frame" />
+    <origin xyz="0.442 0 -1.5167" rpy="0 0 0" />
   </joint>
-  <link name="imu_link"> </link>
+  <link name="imu"> </link>
   <joint name="imu_joint" type="fixed">
-    <parent link="chassis_link" />
-    <child link="imu_link" />
-    <origin xyz="0 0 0" rpy="0 0 0" />
+    <parent link="base_link" />
+    <child link="imu" />
+    <origin xyz="0.442 0 -1.5167" rpy="0 0 0" />
   </joint>
-  <link name="velodyne"> </link>
-  <joint name="velodyne_joint" type="fixed">
-    <parent link="chassis_link" />
-    <child link="velodyne" />
+  <link name="laser_link"> </link>
+  <joint name="laser_link" type="fixed">
+    <parent link="base_link" />
+    <child link="laser_link" />
     <origin xyz="0 0 0" rpy="0 0 0" />
   </joint>
   <link name="navsat_link"> </link>
   <joint name="navsat_joint" type="fixed">
-    <parent link="chassis_link" />
+    <parent link="base_link" />
     <child link="navsat_link" />
     <origin xyz="0 0 0" rpy="0 0 0" />

Commit message: 将imu与baselink固定

File: launch/include/config/robot.urdf.xacro (robot description, xacro)
@@ -7,5 +7,5 @@
     <parent link="base_link"/>
     <child link="base_frame" />
-    <origin xyz="0.442 0 -1.5167" rpy="0 0 0" />
+    <origin xyz="0 0 0" rpy="0 0 0" />
   </joint>
   <link name="imu"> </link>
@@ -13,5 +13,5 @@
     <parent link="base_link" />
     <child link="imu" />
-    <origin xyz="0.442 0 -1.5167" rpy="0 0 0" />
+    <origin xyz="0 0 0" rpy="0 0 0" />
   </joint>
   <link name="laser_link"> </link>
@@ -19,5 +19,5 @@
     <parent link="base_link" />
     <child link="laser_link" />
-    <origin xyz="0 0 0" rpy="0 0 0" />
+    <origin xyz="-0.442 0 1.5167" rpy="0 0 0" />
   </joint>
   <link name="navsat_link"> </link>

Commit message: 程序中对于imu加速度输入先乘以9.8

File: launch/include/config/robot.urdf.xacro (robot description, xacro)
@@ -13,5 +13,5 @@
     <parent link="base_link" />
     <child link="imu" />
-    <origin xyz="0.442 0 -1.5167" rpy="0 0 0" />
+    <origin xyz="0.0 0 0.044" rpy="0 0 0" />
   </joint>
   <link name="laser_link"> </link>

Commit message: 适配车载imu

File: launch/include/config/robot.urdf.xacro (robot description, xacro)
@@ -7,5 +7,5 @@
     <parent link="base_link"/>
     <child link="base_frame" />
-    <origin xyz="0.442 0 -1.5167" rpy="0 0 0" />
+    <origin xyz="0.45 0.0 -0.3" rpy="0 0 0" />
   </joint>
   <link name="imu"> </link>
@@ -13,5 +13,5 @@
     <parent link="base_link" />
     <child link="imu" />
-    <origin xyz="0.0 0 0.044" rpy="0 0 0" />
+    <origin xyz="0.45 0.0 -0.3" rpy="0 0 0" />
   </joint>
   <link name="laser_link"> </link>
@@ -21,9 +21,9 @@
     <origin xyz="0 0 0" rpy="0 0 0" />
   </joint>
-  <link name="navsat_link"> </link>
+<!--  <link name="navsat_link"> </link>
   <joint name="navsat_joint" type="fixed">
     <parent link="base_link" />
     <child link="navsat_link" />
     <origin xyz="0 0 0" rpy="0 0 0" />
-  </joint>
+  </joint>-->
 </robot>

Commit message: 适配改装车tf

File: launch/include/config/robot.urdf.xacro (robot description, xacro)
@@ -7,5 +7,5 @@
     <parent link="base_link"/>
     <child link="base_frame" />
-    <origin xyz="0.45 0.0 -0.3" rpy="0 0 0" />
+    <origin xyz="0.40501 -0.015 -0.231" rpy="0 0 0" />
   </joint>
   <link name="imu"> </link>
@@ -13,5 +13,5 @@
     <parent link="base_link" />
     <child link="imu" />
-    <origin xyz="0.45 0.0 -0.3" rpy="0 0 0" />
+    <origin xyz="0.40501 -0.015 -0.231" rpy="0 0 0" />
   </joint>
   <link name="laser_link"> </link>
